File: Hardware/Schema/SolarPoints/SolarPoints.kicad_sch (KiCad schematic)
At the start: 0 parts

Commit message: update
Other:
- added sheet sheet_1_Power Management (sheet_1_Power Management.kicad_sch)
- added sheet sheet_2_Batteries (sheet_2_Batteries.kicad_sch)
- added sheet sheet_3_Battery Managemen... (sheet_3_Battery Management.kicad_sch)
- added sheet sheet_4_Switching DC-DC C... (sheet_4_Switching DC-DC Conversion.kicad_sch)
- added sheet sheet_5_Microcontroller (sheet_5_Microcontroller.kicad_sch)
- title: (none) -> Cover
Changed lines of the file:
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@@
-(kicad_sch
-	(version 20250114)
-	(generator "eeschema")
-	(generator_version "9.0")
-	(paper "A4")
-	(sheet_instances
-		(path "/"
-			(page "1")
-		)
-	)
-	(embedded_fonts no)
+(kicad_sch (version 20230121) (generator CELUS)
+  (paper "A3")
+  (junction (at 59.07 20.32) (diameter 0)
+  )
+  (bus_entry (at 53.99 26.67) (size 2.54 2.54)
+    (stroke (width 0) (type default))
+  )
+  (bus_entry (at 53.99 41.91) (size 2.54 2.54)
+    (stroke (width 0) (type default))
+  )
+  (wire (pts (xy 34.94 26.67) (xy 53.99 26.67))
+  )
+  (wire (pts (xy 34.94 41.91) (xy 53.99 41.91))
+  )
+  (bus (pts (xy 56.53 22.86) (xy 56.53 44.45))
+  )
+  (bus (pts (xy 56.53 22.86) (xy 59.07 20.32))
+  )
+  (bus (pts (xy 59.07 20.32) (xy 59.07 20.32))
+  )
+  (label "GPIO4" (at 37.48 26.67 0)
+    (effects (justify left bottom))
+  )
+  (label "GPIO4" (at 37.48 41.91 0)
+    (effects (justify left bottom))
+  )
+  (sheet (at 25.4 25.4) (size 9.54 2.54)
+    (stroke (width 0.1524) (type solid) (color 0 0 0 0))
+    (fill (type background) (color 255 255 194 1.0000))
+    (property "Sheetname" "sheet_1_Power Management" (at 25.4 22.86 0)
+      (effects (justify left))
+    )
+    (property "Sheetfile" "sheet_1_Power Management.kicad_sch" (at 25.4 29.21 0)
+      (effects hide)
+    )
+    (pin "GPIO4" bidirectional (at 34.94 26.67 0)
+      (effects (font (size 1.27 1.27)) (justify right))
+    )
+  )
+  (sheet (at 25.4 33.02) (size 9.54 2.54)
+    (stroke (width 0.1524) (type solid) (color 0 0 0 0))
+    (fill (type background) (color 255 255 194 1.0000))
+    (property "Sheetname" "sheet_2_Batteries" (at 25.4 30.48 0)
+      (effects (justify left))
+    )
+    (property "Sheetfile" "sheet_2_Batteries.kicad_sch" (at 25.4 36.83 0)
+      (effects hide)
+    )
+  )
+  (sheet (at 25.4 40.64) (size 9.54 2.54)
+    (stroke (width 0.1524) (type solid) (color 0 0 0 0))
+    (fill (type background) (color 255 255 194 1.0000))
+    (property "Sheetname" "sheet_3_Battery Managemen..." (at 25.4 38.1 0)
+      (effects (justify left))
+    )
+    (property "Sheetfile" "sheet_3_Battery Management.kicad_sch" (at 25.4 44.45 0)
+      (effects hide)
+    )
+    (pin "GPIO4" bidirectional (at 34.94 41.91 0)
+      (effects (font (size 1.27 1.27)) (justify right))
+    )
+  )
+  (sheet (at 25.4 48.26) (size 9.54 2.54)
+    (stroke (width 0.1524) (type solid) (color 0 0 0 0))
+    (fill (type background) (color 255 255 194 1.0000))
+    (property "Sheetname" "sheet_4_Switching DC-DC C..." (at 25.4 45.72 0)
+      (effects (justify left))
+    )
+    (property "Sheetfile" "sheet_4_Switching DC-DC Conversion.kicad_sch" (at 25.4 52.07 0)
+      (effects hide)
+    )
+  )
+  (sheet (at 25.4 55.88) (size 9.54 2.54)
+    (stroke (width 0.1524) (type solid) (color 0 0 0 0))
+    (fill (type background) (color 255 255 194 1.0000))
+    (property "Sheetname" "sheet_5_Microcontroller" (at 25.4 53.34 0)
+      (effects (justify left))
+    )
+    (property "Sheetfile" "sheet_5_Microcontroller.kicad_sch" (at 25.4 59.69 0)
+      (effects hide)
+    )
+  )
+  (title_block
+    (date "2025/10/09")
+    (title "Cover")
+    (rev "0")
+    (comment 1 "https://www.celus.io/terms-of-use-celus-design-platform")
+    (comment 2 "fegrolla0210@gmail.com")
+    (comment 3 "default_project_name_1756300784107")
+  )
 )
